File: eGPU-dock/eGPU-dock.kicad_sch (KiCad schematic)
At the start: 7 parts, among them J1 Bus_M.2_Socket_M, U1 X1611WVS-164-9TV30, U3 CYUSB3304-68LTXC_C462531, U4 CYUSB3304-68LTXC_C462531

Commit message: update kicad
Parts:
- removed J1: Bus_M.2_Socket_M, symbol Connector:Bus_M.2_Socket_M
- removed U3, U4: CYUSB3304-68LTXC_C462531, easyeda2kicad:QFN-68_L8.0-W8.0-P0.40-BL-EP5.1, symbol easyeda2kicad:CYUSB3304-68LTXC_C462531
- removed USB1, USB2: TYPE-C 24P QCHT, easyeda2kicad:TYPE-C-SMD_TYPE-C-24P-QCHT, symbol easyeda2kicad:TYPE-C24PQCHT
- added ASM2: ~, easyeda2kicad:FCCSP-273_L10.0-W10.0-P0.45-TL, symbol easyeda2kicad:ASM2464PD
- added C1: 10p, Capacitor_SMD:C_0402_1005Metric, symbol Device:C_Small
- added C2, C3, C4, C5, C6, C7, C8, C9: 0.33u, Capacitor_SMD:C_0201_0603Metric, symbol Device:C_Small
- added HUB1: CYUSB4347-BZXC, easyeda2kicad:FBGA-192_L12.0-W12.0-P0.80-BL_CY9BF318TBGL-GK7E1, symbol easyeda2kicad:CYUSB4347-BZXC
- added NVME1: AS0BC21-S40BM-7H, easyeda2kicad:CONN-SMD_AS0BC21-S40BM-7H, symbol easyeda2kicad:AS0BC21-S40BM-7H
- added R3, R4, R5, R6, R7, R8: 0Ω, Resistor_SMD:R_0402_1005Metric, symbol Device:R_Small
- added USB1, USB2, USB3, USB4, USB5: USB_C_Receptacle, easyeda2kicad:USB-C-TH_12401832E402A, symbol Connector:USB_C_Receptacle
- added USB6, USB7: USB3_A, Connector_USB:USB3_A_Molex_48393-001, symbol Connector:USB3_A
- added USB8, USB9: USB_A, Connector_USB:USB_A_Molex_67643_Horizontal, symbol Connector:USB_A
- added Y1: 25MHz, Crystal:Crystal_SMD_3225-4Pin_3.2x2.5mm, symbol Device:Crystal_GND24
- ASM1: renamed from U2; footprint ProLib_pcs_2025-11-17:FCCSP-273_L10.0-W10.0-P0.45-TL -> easyeda2kicad:FCCSP-273_L10.0-W10.0-P0.45-TL
- renumbered U1 to PCIe1
Connections:
- net ActLED2: now reaches ASM1.A1 (GPIO3)
- net GPIO19: now reaches ASM1.A10 (GPIO19)
- net GPIO20: now reaches ASM1.A11 (GPIO20)
- net GPIO21: now reaches ASM1.A12 (GPIO21)
- net PE_WAKE#: now reaches ASM1.A13 (GPIO22)
- net CLKREQ2#: now reaches ASM1.A14 (GPIO23)
- net CLKREQ3#: now reaches ASM1.A15 (GPIO24)
- net ActLED3: now reaches ASM1.A16 (GPIO25)
- net ActLED4: now reaches ASM1.A17 (GPIO26)
- net GPIO27: now reaches ASM1.A18 (GPIO27)
- net CLKREQ1#: now reaches ASM1.A19 (GPIO8)
- net SPI_CS#: now reaches ASM1.A2 (SPI_CS#)
- net CLKREQ0#: now reaches ASM1.A20 (GPIO14)
- net UART_RX: now reaches ASM1.A21 (UART_RX)
- net SPI_DO: now reaches ASM1.A3 (SPI_DO)
- net SPI_DI: now reaches ASM1.A4 (SPI_DI)
- net SPI_CLK: now reaches ASM1.A5 (SPI_CLK)
- net P1_LED: now reaches ASM1.A6 (GPIO15)
- net P2_LED: now reaches ASM1.A7 (GPIO16)
- net P3_LED: now reaches ASM1.A8 (GPIO17)
- net P4_LED: now reaches ASM1.A9 (GPIO18)
- net PCIe_RX3+: now reaches ASM1.AA13 (PRXP3)
- net PCIe_TX3-: now reaches ASM1.AA15 (PTXN3)
- net PCIe_TX2-: now reaches ASM1.AA17 (PTXN2)
- net PCIe_RX2-: now reaches ASM1.AA19 (PRXN2)
- net CC1: now reaches ASM1.AA6 (CC1)
- net CC1: now also R3.2
- net REFCLK+: now reaches ASM1.AA8 (REFCLKP0)
- net GPIO2: now reaches ASM1.B1 (GPIO2)
- net UART_TX: now reaches ASM1.B21 (UART_TX)
- net GPIO1: now reaches ASM1.C1 (GPIO1)
- net HDDPC: now reaches ASM1.C21 (HDDPC)
- net ActLED1: now reaches ASM1.D1 (GPIO0)
- net I2C_CLK: now reaches ASM1.E1 (I2C_CLK_P)
- net I2C_DATA: now reaches ASM1.F1 (I2C_DATA_P)
- net VBUS: now reaches ASM1.G1 (VBUS)
- net PERST0#: now reaches ASM1.G21 (PERST0#)
- net RST#: now reaches ASM1.H1 (RST#)
- net TEST_EN: now reaches ASM1.H21 (TEST_EN)
- net SBU2: now reaches ASM1.J1 (SBU2)
- net SBU2: now also R8.2
- net SBU1: now reaches ASM1.K1 (SBU1)
- net SBU1: now also R7.2
- net USB2_D+: now reaches ASM1.M1 (UDP)
- net USB2_D+: now also R6.2
- net USB2_D-: now reaches ASM1.M2 (UDM)
- net USB2_D-: now also R5.2
- net PCIe_RX0-: now reaches ASM1.N20 (PRXN0)
- net PCIe_RX0+: now reaches ASM1.N21 (PRXP0)
- net URX0+: now reaches ASM1.P1 (URXP0)
- net URX0+: now also C3.2
- net URX0-: now reaches ASM1.P2 (URXN0)
- net URX0-: now also C2.2
- net PCIe_TX0+: now reaches ASM1.R20 (PTXP0)
- net PCIe_TX0-: now reaches ASM1.R21 (PTXN0)
- net UTX0+: now reaches ASM1.T1 (UTXP0)
- net UTX0+: now also C5.2
- net UTX0-: now reaches ASM1.T2 (UTXN0)
- net UTX0-: now also C4.2
- net PCIe_TX1+: now reaches ASM1.U20 (PTXP1)
- net PCIe_TX1-: now reaches ASM1.U21 (PTXN1)
- net UTX1-: now reaches ASM1.V1 (UTXN1)
- net UTX1-: now also C8.2
- net UTX1+: now reaches ASM1.V2 (UTXP1)
- net UTX1+: now also C9.2
- net PCIe_RX1-: now reaches ASM1.W20 (PRXN1)
- net PCIe_RX1+: now reaches ASM1.W21 (PRXP1)
- net URX1-: now reaches ASM1.Y1 (URXN1)
- net URX1-: now also C6.2
- net PCIe_RX3-: now reaches ASM1.Y13 (PRXN3)
- net PCIe_TX3+: now reaches ASM1.Y15 (PTXP3)
- net PCIe_TX2+: now reaches ASM1.Y17 (PTXP2)
- net PCIe_RX2+: now reaches ASM1.Y19 (PRXP2)
- net URX1+: now reaches ASM1.Y2 (URXP1)
- net URX1+: now also C7.2
- net CC2: now reaches ASM1.Y6 (CC2)
- net CC2: now also R4.2
- net REFCLK-: now reaches ASM1.Y8 (REFCLKN0)
- net UREXT: now reaches ASM1.AA3 (REXT)
- net XI: now reaches ASM1.AA4 (XI)
- net XI: now also C1.2, Y1.3
- net XO: now reaches ASM1.Y4 (XO)
- net XO: now also C1.1, Y1.1
- new net: USB3.A1 (GND), USB3.A12 (GND), USB3.B1 (GND), USB3.B12 (GND)
- new net: USB3.A4 (VBUS), USB3.A9 (VBUS), USB3.B4 (VBUS), USB3.B9 (VBUS)
- new net: USB5.A1 (GND), USB5.A12 (GND), USB5.B1 (GND), USB5.B12 (GND)
- new net: USB5.A4 (VBUS), USB5.A9 (VBUS), USB5.B4 (VBUS), USB5.B9 (VBUS)
- new net: USB2.A1 (GND), USB2.A12 (GND), USB2.B1 (GND), USB2.B12 (GND)
- new net: USB2.A4 (VBUS), USB2.A9 (VBUS), USB2.B4 (VBUS), USB2.B9 (VBUS)
- new net: USB4.A1 (GND), USB4.A12 (GND), USB4.B1 (GND), USB4.B12 (GND)
- new net: USB4.A4 (VBUS), USB4.A9 (VBUS), USB4.B4 (VBUS), USB4.B9 (VBUS)
- new net +5V_VBUS: USB1.A4 (VBUS), USB1.A9 (VBUS), USB1.B4 (VBUS), USB1.B9 (VBUS)
- new net CC1_C: R3.1, USB1.A5 (CC1)
- new net CC2_C: R4.1, USB1.B5 (CC2)
- new net GND: USB1.A1 (GND), USB1.A12 (GND), USB1.B1 (GND), USB1.B12 (GND), USB1.S1 (SHIELD), Y1.2, Y1.4
- new net SBU1_C: R7.1, USB1.A8 (SBU1)
- new net SBU2_C: R8.1, USB1.B8 (SBU2)
- new net URX0_C+: C3.1, USB1.B11 (RX1+)
- new net URX0_C-: C2.1, USB1.B10 (RX1-)
- new net URX1_C+: C7.1, USB1.A11 (RX2+)
- new net URX1_C-: C6.1, USB1.A10 (RX2-)
- new net USB2_C_D+: R6.1, USB1.A6 (D+), USB1.B6 (D+)
- new net USB2_C_D-: R5.1, USB1.A7 (D-), USB1.B7 (D-)
- new net UTX0_C+: C5.1, USB1.A2 (TX1+)
- new net UTX0_C-: C4.1, USB1.A3 (TX1-)
- new net UTX1_C+: C9.1, USB1.B2 (TX2+)
- new net UTX1_C-: C8.1, USB1.B3 (TX2-)
- no-connect marks 0 -> 41
Other:
- note added: "0201 for USB4"
- moved on the sheet: ASM1B, PCIe1

Commit message: update kicad
Parts:
- added C10, C11, C12, C13, C14, C15, C16, C17, C18, C19, C20, C21, C22, C23, C24, C25: 0.22u, Capacitor_SMD:C_0402_1005Metric, symbol Device:C_Small
- added J1: Bus_PCI_Express_x16, Connector_PCBEdge:BUS_PCIexpress_x16, symbol Connector:Bus_PCI_Express_x16
- added J2: PCIexpress_x16, PCIexpress:PCIexpress_x16, symbol egpulib:PCIexpress_x16
- added R1, R2, R30, R31, R9: 0Ω, Resistor_SMD:R_0402_1005Metric, symbol Device:R_Small
- USB1, USB2, USB3, USB4, USB5: footprint easyeda2kicad:USB-C-TH_12401832E402A -> Connector_USB:USB_C_Receptacle_Amphenol_12401610E4-2A
Connections:
- net CLKREQ0#: now also R1.1, R30.2
- net GND: now also PCIe1.B4, J1.A1 (~{PRSNT1}), J1.A12 (GND), J1.A15 (GND), J1.A18 (GND), J1.A20 (GND), J1.A23 (GND), J1.A24 (GND), J1.A27 (GND), J1.A28 (GND), J1.A31 (GND), J1.A34 (GND), J1.A37 (GND), J1.A38 (GND), J1.A4 (GND), J1.A41 (GND), J1.A42 (GND), J1.A45 (GND), J1.A46 (GND), J1.A49 (GND), J1.A51 (GND), J1.A54 (GND), J1.A55 (GND), J1.A58 (GND), J1.A59 (GND), J1.A62 (GND), J1.A63 (GND), J1.A66 (GND), J1.A67 (GND), J1.A70 (GND), J1.A71 (GND), J1.A74 (GND), J1.A75 (GND), J1.A78 (GND), J1.A79 (GND), J1.A82 (GND), J1.B13 (GND), J1.B16 (GND), J1.B18 (GND), J1.B21 (GND), J1.B22 (GND), J1.B25 (GND), J1.B26 (GND), J1.B29 (GND), J1.B32 (GND), J1.B35 (GND), J1.B36 (GND), J1.B39 (GND), J1.B4 (GND), J1.B40 (GND), J1.B43 (GND), J1.B44 (GND), J1.B47 (GND), J1.B49 (GND), J1.B52 (GND), J1.B53 (GND), J1.B56 (GND), J1.B57 (GND), J1.B60 (GND), J1.B61 (GND), J1.B64 (GND), J1.B65 (GND), J1.B68 (GND), J1.B69 (GND), J1.B7 (GND), J1.B72 (GND), J1.B73 (GND), J1.B76 (GND), J1.B77 (GND), J1.B80 (GND), R9.1
- net PCIe_RX0+: now also PCIe1.A16, J2.A16 (PERp0)
- net PCIe_RX0-: now also PCIe1.A17, J2.A17 (PERn0)
- net PCIe_RX1+: now also PCIe1.A21, J2.A21 (PERp1)
- net PCIe_RX1-: now also PCIe1.A22, J2.A22 (PERn1)
- net PCIe_RX2+: now also PCIe1.A25, J2.A25 (PERp2)
- net PCIe_RX2-: now also PCIe1.A26, J2.A26 (PERn2)
- net PCIe_RX3+: now also PCIe1.A29, J2.A29 (PERp3)
- net PCIe_RX3-: now also PCIe1.A30, J2.A30 (PERn3)
- net PCIe_TX0+: now also C10.1, C12.1
- net PCIe_TX0-: now also C11.1, C13.1
- net PCIe_TX1+: now also C14.1, C20.1
- net PCIe_TX1-: now also C15.1, C21.1
- net PCIe_TX2+: now also C16.1, C22.1
- net PCIe_TX2-: now also C17.1, C23.1
- net PCIe_TX3+: now also C18.1, C24.1
- net PCIe_TX3-: now also C19.1, C25.1
- net PERST0#: now also PCIe1.A11, J1.A11 (~{PERST})
- net PE_WAKE#: now also R2.1, R31.1
- net REFCLK+: now also PCIe1.A13, J1.A13 (REFCLK+)
- net REFCLK-: now also PCIe1.A14, J1.A14 (REFCLK-)
- net at PCIe1.165: now also PCIe1.A12, PCIe1.A15, PCIe1.A18, PCIe1.A20, PCIe1.A23, PCIe1.A24, PCIe1.A27, PCIe1.A28, PCIe1.A31, PCIe1.A34, PCIe1.A37, PCIe1.A38, PCIe1.A4, PCIe1.A41, PCIe1.A42, PCIe1.A45, PCIe1.A46, PCIe1.A49, PCIe1.A51, PCIe1.A54, PCIe1.A55, PCIe1.A58, PCIe1.A59, PCIe1.A62, PCIe1.A63, PCIe1.A66, PCIe1.A67, PCIe1.A70, PCIe1.A71, PCIe1.A74, PCIe1.A75, PCIe1.A78, PCIe1.A79, PCIe1.A82
- net at PCIe1.B11: now also R31.2
- net PCIe_TX0_C+: now reaches PCIe1.B14
- net PCIe_TX0_C+: now also C10.2, C12.2, J2.B14 (PETp0)
- net PCIe_TX0_C-: now reaches PCIe1.B15
- net PCIe_TX0_C-: now also C11.2, C13.2, J2.B15 (PETn0)
- net at PCIe1.B17: now also PCIe1.B31, R30.1
- net PCIe_TX1_C+: now reaches PCIe1.B19
- net PCIe_TX1_C+: now also C14.2, C20.2, J2.B19 (PETp1)
- net PCIe_TX1_C-: now reaches PCIe1.B20
- net PCIe_TX1_C-: now also C15.2, C21.2, J2.B20 (PETn1)
- net PCIe_TX2_C+: now reaches PCIe1.B23
- net PCIe_TX2_C+: now also C16.2, C22.2, J2.B23 (PETp2)
- net PCIe_TX2_C-: now reaches PCIe1.B24
- net PCIe_TX2_C-: now also C17.2, C23.2, J2.B24 (PETn2)
- net PCIe_TX3_C+: now reaches PCIe1.B27
- net PCIe_TX3_C+: now also C18.2, C24.2, J2.B27 (PETp3)
- net PCIe_TX3_C-: now reaches PCIe1.B28
- net PCIe_TX3_C-: now also C19.2, C25.2, J2.B28 (PETn3)
- net Card_SMBCLK: now reaches PCIe1.B5
- net Card_SMBCLK: now also J1.B5 (SMCLK)
- net Card_SMBDAT: now reaches PCIe1.B6
- net Card_SMBDAT: now also J1.B6 (SMDAT)
- new net: J2.A1 (~{PRSNT1}), R9.2
- new net: J1.B17 (~{PRSNT2}), J1.B31 (~{PRSNT2}), J1.B48 (~{PRSNT2}), J1.B81 (~{PRSNT2}), R1.2
- new net: J1.A2 (+12V), J1.A3 (+12V), J1.B1 (+12V), J1.B2 (+12V), J1.B3 (+12V)
- new net: J1.B11 (~{WAKE}), R2.2
- new net: J2.A12 (GND), J2.A15 (GND), J2.A18 (GND), J2.A20 (GND), J2.A23 (GND), J2.A24 (GND), J2.A27 (GND), J2.A28 (GND), J2.A31 (GND), J2.A34 (GND), J2.A37 (GND), J2.A38 (GND), J2.A4 (GND), J2.A41 (GND), J2.A42 (GND), J2.A45 (GND), J2.A46 (GND), J2.A49 (GND), J2.A51 (GND), J2.A54 (GND), J2.A55 (GND), J2.A58 (GND), J2.A59 (GND), J2.A62 (GND), J2.A63 (GND), J2.A66 (GND), J2.A67 (GND), J2.A70 (GND), J2.A71 (GND), J2.A74 (GND), J2.A75 (GND), J2.A78 (GND), J2.A79 (GND), J2.A82 (GND)
- new net: J2.B13 (GND), J2.B16 (GND), J2.B18 (GND), J2.B21 (GND), J2.B22 (GND), J2.B25 (GND), J2.B26 (GND), J2.B29 (GND), J2.B32 (GND), J2.B35 (GND), J2.B36 (GND), J2.B39 (GND), J2.B4 (GND), J2.B40 (GND), J2.B43 (GND), J2.B44 (GND), J2.B47 (GND), J2.B49 (GND), J2.B52 (GND), J2.B53 (GND), J2.B56 (GND), J2.B57 (GND), J2.B60 (GND), J2.B61 (GND), J2.B64 (GND), J2.B65 (GND), J2.B68 (GND), J2.B69 (GND), J2.B7 (GND), J2.B72 (GND), J2.B73 (GND), J2.B76 (GND), J2.B77 (GND), J2.B80 (GND)
- new net +12V_PCIe: J2.A2 (+12V), J2.A3 (+12V), J2.B1 (+12V), J2.B2 (+12V), J2.B3 (+12V)
- new net +3.3V_PCIe: J1.A10 (+3.3V), J1.A9 (+3.3V), J1.B10 (3.3Vaux), J1.B8 (+3.3V)
Other:
- moved on the sheet: PCIe1

Commit message: update
Parts:
- removed C12, C13, C14, C15, C16, C17, C18, C19: 0.22u, Capacitor_SMD:C_0402_1005Metric, symbol Device:C_Small
- removed PCIe1: X1611WVS-164-9TV30, easyeda2kicad:CONN-SMD_164P-P1.00_X1611WVS-164-9TV30, symbol easyeda2kicad:X1611WVS-164-9TV30
- removed R30, R31: 0Ω, Resistor_SMD:R_0402_1005Metric, symbol Device:R_Small
- added R10, R11, R12, R13, R14, R15, R16, R17, R18, R19, R20, R21, R22: 0Ω, Resistor_SMD:R_0402_1005Metric, symbol Device:R_Small
- added R23: 4.7kΩ, Resistor_SMD:R_0402_1005Metric, symbol Device:R_Small
- PCIe1: renamed from J2; footprint PCIexpress:PCIexpress_x16 -> easyeda2kicad:CONN-SMD_164P-P1.00_X1611WVS-164-9TV30
Connections:
- net +3.3V_PCIe: now also PCIe1.A10 (+3.3V), PCIe1.A9 (+3.3V), PCIe1.B8 (+3.3V)
- net Card_SMBDAT: now also R10.1; no longer J1.B6 (SMDAT)
- net PCIe_RX0+: now also R14.2; no longer PCIe1.A16 (PERp0)
- net PCIe_RX0-: now also R15.2; no longer PCIe1.A17 (PERn0)
- net PCIe_RX1+: now also R16.2; no longer PCIe1.A21 (PERp1)
- net PCIe_RX1-: now also R17.2; no longer PCIe1.A22 (PERn1)
- net PCIe_RX2+: now also R18.2; no longer PCIe1.A25 (PERp2)
- net PCIe_RX2-: now also R19.2; no longer PCIe1.A26 (PERn2)
- net PCIe_RX3+: now also R20.2; no longer PCIe1.A29 (PERp3)
- net PCIe_RX3-: now also R21.2; no longer PCIe1.A30 (PERn3)
- net REFCLK+: no longer J1.A13 (REFCLK+)
- net REFCLK-: no longer J1.A14 (REFCLK-)
- net PCIe_PRSNT1: now reaches PCIe1.A1 (~{PRSNT1}), R9.2
- net at J1.B11 (~{WAKE}): no longer R2.2
- net at PCIe1.A13 (REFCLK+): now also R12.1
- net at PCIe1.A14 (REFCLK-): now also R13.1
- net +3.3V_aux: now reaches PCIe1.B10 (+3.3V_aux)
- net at PCIe1.B11 (~{WAKE}): now also R2.2
- net at PCIe1.B17 (~{PRSNT2}): now also R22.2, R23.2
- net at PCIe1.B5 (SMCLK): now also R11.2
- net at PCIe1.B6 (SMDAT): now also R10.2
- net Card_SMBCLK: no longer names the net of J1.B5 (SMCLK)
- new net: PCIe1.A17 (PERn0), R15.1
- new net: PCIe1.A22 (PERn1), R17.1
- new net: PCIe1.A26 (PERn2), R19.1
- new net: PCIe1.A30 (PERn3), R21.1
- new net: PCIe1.A16 (PERp0), R14.1
- new net: PCIe1.A21 (PERp1), R16.1
- new net: PCIe1.A25 (PERp2), R18.1
- new net: PCIe1.A29 (PERp3), R20.1
- new net +3.3V: R23.1
- new net PCIe_REFCLK+: R12.2
- new net PCIe_REFCLK-: R13.2
- new net PCIe_SMCLK: R11.1
Other:
- moved on the sheet: R2, R9

Commit message: finish symbol and footprint
Parts:
- removed J1: Bus_PCI_Express_x16, Connector_PCBEdge:BUS_PCIexpress_x16, symbol Connector:Bus_PCI_Express_x16
- removed R1: 0Ω, Resistor_SMD:R_0402_1005Metric, symbol Device:R_Small
- added GbE1: AQR113C/AQR114C/AQR115C, eGPUlib:AQR113C-AQR114C-AQR115C, symbol egpulib:AQR113C-AQR114C-AQR115C_1_1
Other:
- moved on the sheet: NVME1

Commit message: stuff
Parts:
- added HUB2: CYUSB4347-BZXC, easyeda2kicad:FBGA-192_L12.0-W12.0-P0.80-BL_CY9BF318TBGL-GK7E1, symbol easyeda2kicad:CYUSB4347-BZXC
- added NVME2: AS0BC21-S40BM-7H, easyeda2kicad:CONN-SMD_AS0BC21-S40BM-7H, symbol easyeda2kicad:AS0BC21-S40BM-7H
- added USB10, USB11: USB_C_Receptacle, Connector_USB:USB_C_Receptacle_Amphenol_12401610E4-2A, symbol Connector:USB_C_Receptacle
- added USB12, USB13: USB_A, Connector_USB:USB_A_Molex_67643_Horizontal, symbol Connector:USB_A
Connections:
- new net: USB10.A1 (GND), USB10.A12 (GND), USB10.B1 (GND), USB10.B12 (GND)
- new net: USB10.A4 (VBUS), USB10.A9 (VBUS), USB10.B4 (VBUS), USB10.B9 (VBUS)
- new net: USB11.A1 (GND), USB11.A12 (GND), USB11.B1 (GND), USB11.B12 (GND)
- new net: USB11.A4 (VBUS), USB11.A9 (VBUS), USB11.B4 (VBUS), USB11.B9 (VBUS)
