File: eGPU-dock/eGPU-dock.kicad_sch (KiCad schematic)
At the start: 55 parts, among them Y1 25MHz

Commit message: add diagram and stuff
Parts:
- added HUB2: CYUSB4347-BZXC, easyeda2kicad:FBGA-192_L12.0-W12.0-P0.80-BL_CY9BF318TBGL-GK7E1, symbol easyeda2kicad:CYUSB4347-BZXC
- added SD1: GL3232S-ONY04, easyeda2kicad:QFN-48_L6.0-W6.0-P0.40-TL-EP4.5, symbol easyeda2kicad:GL3232S-ONY04

Commit message: update
Parts:
- removed ASM1, ASM2: ~, easyeda2kicad:FCCSP-273_L10.0-W10.0-P0.45-TL, symbol easyeda2kicad:ASM2464PD
- removed GbE1: AQR113C/AQR114C/AQR115C, eGPUlib:AQR113C-AQR114C-AQR115C, symbol egpulib:AQR113C-AQR114C-AQR115C_1_1
- removed HUB1, HUB2: CYUSB4347-BZXC, easyeda2kicad:FBGA-192_L12.0-W12.0-P0.80-BL_CY9BF318TBGL-GK7E1, symbol easyeda2kicad:CYUSB4347-BZXC
- removed R19, R20: 0Ω, Resistor_SMD:R_0402_1005Metric, symbol Device:R_Small
- removed R23: 4.7kΩ, Resistor_SMD:R_0402_1005Metric, symbol Device:R_Small
- removed SD1: GL3232S-ONY04, easyeda2kicad:QFN-48_L6.0-W6.0-P0.40-TL-EP4.5, symbol easyeda2kicad:GL3232S-ONY04
- removed USB6, USB7: USB3_A, Connector_USB:USB3_A_Molex_48393-001, symbol Connector:USB3_A
- removed USB8, USB9: USB_A, Connector_USB:USB_A_Molex_67643_Horizontal, symbol Connector:USB_A
- removed Y1: 25MHz, Crystal:Crystal_SMD_3225-4Pin_3.2x2.5mm, symbol Device:Crystal_GND24
- added ASM1, ASM2: ~, eGPUlib:ASM2464PDX, symbol egpulib:ASM2464PDX
- added C12, C13, C14, C15, C16, C17, C18: 0.33u, Capacitor_SMD:C_0201_0603Metric, symbol Device:C_Small
- added C19, C26, C27, C28: 0.22u, Capacitor_SMD:C_0402_1005Metric, symbol Device:C_Small
- added C29: 220p, Capacitor_SMD:C_0402_1005Metric, symbol Device:C_Small
- added R1: 10k, Resistor_SMD:R_0402_1005Metric, symbol Device:R_Small
- added U1: PCI11414-I/PMX, easyeda2kicad:QFN-164_L13.0-W13.0-P0.50-TL-EP8.0, symbol easyeda2kicad:PCI11414-I_PMX
- added U2: USB7216C/KDX, easyeda2kicad:VQFN-100_L12.0-W12.0-P0.40-TL-EP8.0, symbol easyeda2kicad:USB7216C_KDX
- added U3: USB7206C-I/KDX, easyeda2kicad:VQFN-100_L12.0-W12.0-P0.40-TL-EP8.0, symbol easyeda2kicad:USB7206C-I_KDX
- added USB10, USB7, USB8, USB9: HC-USB3.0-L257-P, easyeda2kicad:USB-3.0-A-TH_HOOYA_USB-303L-L-SU, symbol easyeda2kicad:HC-USB3.0-L257-P
- added USB11, USB12: USB-269-BRW, easyeda2kicad:USB-A-TH_USB-269-BRW, symbol easyeda2kicad:USB-269-BRW
- added USB6: USB_C_Receptacle, Connector_USB:USB_C_Receptacle_Amphenol_12401610E4-2A, symbol Connector:USB_C_Receptacle
- C1: value 10p -> 0.33u; footprint Capacitor_SMD:C_0402_1005Metric -> Capacitor_SMD:C_0201_0603Metric
- R15, R16, R21: value 0Ω -> 10k
- R17: value 0Ω -> 1KΩ
- R18: value 0Ω -> 10KΩ
Connections:
- net Card_SMBDAT is gone; now on net USB4_2_CC2_C: R10.1
- net PCIe_SMCLK is gone; now on net USB4_2_2.0_C_D-: R11.1
- net XO is gone; now on net USB4_2_RX0_C-: C1.1
- net +5V_VBUS: now also USB2.A4 (VBUS), USB2.A9 (VBUS), USB2.B4 (VBUS), USB2.B9 (VBUS)
- net GND: now also NVME1.1, NVME1.15, NVME1.21, NVME1.27, NVME1.3, NVME1.33, NVME1.39, NVME1.45, NVME1.51, NVME1.57, NVME1.71, NVME1.73, NVME1.75, NVME1.9, PCIe1.A1 (~{PRSNT1}), PCIe1.A12 (GND), PCIe1.A15 (GND), PCIe1.A18 (GND), PCIe1.A20 (GND), PCIe1.A23 (GND), PCIe1.A24 (GND), PCIe1.A27 (GND), PCIe1.A28 (GND), PCIe1.A31 (GND), PCIe1.A34 (GND), PCIe1.A37 (GND), PCIe1.A38 (GND), PCIe1.A4 (GND), PCIe1.A41 (GND), PCIe1.A42 (GND), PCIe1.A45 (GND), PCIe1.A46 (GND), PCIe1.A49 (GND), PCIe1.A51 (GND), PCIe1.A54 (GND), PCIe1.A55 (GND), PCIe1.A58 (GND), PCIe1.A59 (GND), PCIe1.A62 (GND), PCIe1.A63 (GND), PCIe1.A66 (GND), PCIe1.A67 (GND), PCIe1.A70 (GND), PCIe1.A71 (GND), PCIe1.A74 (GND), PCIe1.A75 (GND), PCIe1.A78 (GND), PCIe1.A79 (GND), PCIe1.A82 (GND), PCIe1.B13 (GND), PCIe1.B16 (GND), PCIe1.B18 (GND), PCIe1.B21 (GND), PCIe1.B22 (GND), PCIe1.B25 (GND), PCIe1.B26 (GND), PCIe1.B29 (GND), PCIe1.B32 (GND), PCIe1.B35 (GND), PCIe1.B36 (GND), PCIe1.B39 (GND), PCIe1.B4 (GND), PCIe1.B40 (GND), PCIe1.B43 (GND), PCIe1.B44 (GND), PCIe1.B47 (GND), PCIe1.B49 (GND), PCIe1.B52 (GND), PCIe1.B53 (GND), PCIe1.B56 (GND), PCIe1.B57 (GND), PCIe1.B60 (GND), PCIe1.B61 (GND), PCIe1.B64 (GND), PCIe1.B65 (GND), PCIe1.B68 (GND), PCIe1.B69 (GND), PCIe1.B7 (GND), PCIe1.B72 (GND), PCIe1.B73 (GND), PCIe1.B76 (GND), PCIe1.B77 (GND), PCIe1.B80 (GND), R17.1, USB2.A1 (GND), USB2.A12 (GND), USB2.B1 (GND), USB2.B12 (GND), USB2.S1 (SHIELD), ASM1.D11 (GND), ASM1.D17 (GND), ASM1.D18 (GND), ASM1.D4 (GND), ASM1.D5 (GND), ASM1.E17 (GND), ASM1.E18 (GND), ASM1.E4 (GND), ASM1.E5 (GND), ASM1.F17 (GND), ASM1.F18 (GND), ASM1.F4 (GND), ASM1.F5 (GND), ASM1.F8 (GND), ASM1.H17 (GND), ASM1.H18 (GND), ASM1.H4 (GND), ASM1.H8 (GND), ASM1.J11 (GND), ASM1.J4 (GND), ASM1.J5 (GND), ASM1.J6 (GND), ASM1.K2 (GND), ASM1.L13 (GND), ASM1.L9 (GND), ASM1.N11 (GND), ASM1.N13 (GND), ASM1.N9 (GND), ASM1.P11 (GND), ASM1.P9 (GND), ASM2.D11 (GND), ASM2.D17 (GND), ASM2.D18 (GND), ASM2.D4 (GND), ASM2.D5 (GND), ASM2.E17 (GND), ASM2.E18 (GND), ASM2.E4 (GND), ASM2.E5 (GND), ASM2.F17 (GND), ASM2.F18 (GND), ASM2.F4 (GND), ASM2.F5 (GND), ASM2.F8 (GND), ASM2.H17 (GND), ASM2.H18 (GND), ASM2.H4 (GND), ASM2.H8 (GND), ASM2.J11 (GND), ASM2.J4 (GND), ASM2.J5 (GND), ASM2.J6 (GND), ASM2.K2 (GND), ASM2.L13 (GND), ASM2.L9 (GND), ASM2.N11 (GND), ASM2.N13 (GND), ASM2.N9 (GND), ASM2.P11 (GND), ASM2.P9 (GND), C29.1; no longer R9.1
- net PCIe_REFCLK+: now also PCIe1.A13 (REFCLK+), ASM1.AA8 (REFCLKP0); no longer R12.2
- net PCIe_REFCLK-: now also PCIe1.A14 (REFCLK-), ASM1.Y8 (REFCLKN0); no longer R13.2
- net PCIe_RX0+: now also PCIe1.A16 (PERp0), ASM1.N21 (PRXP0); no longer R14.2
- net PCIe_RX0-: now also PCIe1.A17 (PERn0), ASM1.N20 (PRXN0); no longer R15.2
- net PCIe_RX1+: now also PCIe1.A21 (PERp1), ASM1.W21 (PRXP1); no longer R16.2
- net PCIe_RX1-: now also PCIe1.A22 (PERn1), ASM1.W20 (PRXN1); no longer R17.2
- net PCIe_RX2+: now also PCIe1.A25 (PERp2), ASM1.Y19 (PRXP2); no longer R18.2
- net PCIe_RX2-: now also PCIe1.A26 (PERn2), ASM1.AA19 (PRXN2)
- net PCIe_RX3+: now also PCIe1.A29 (PERp3), ASM1.AA13 (PRXP3)
- net PCIe_RX3-: now also PCIe1.A30 (PERn3), ASM1.Y13 (PRXN3); no longer R21.2
- net PCIe_TX0+: now also ASM1.R20 (PTXP0)
- net PCIe_TX0-: now also ASM1.R21 (PTXN0)
- net PCIe_TX1+: now also ASM1.U20 (PTXP1)
- net PCIe_TX1-: now also ASM1.U21 (PTXN1)
- net PCIe_TX2+: now also ASM1.Y17 (PTXP2)
- net PCIe_TX2-: now also ASM1.AA17 (PTXN2)
- net PCIe_TX3+: now also ASM1.Y15 (PTXP3)
- net PCIe_TX3-: now also ASM1.AA15 (PTXN3)
- net VBUS: now also ASM2.G1 (VBUS)
- net at PCIe1.B6 (SMDAT): no longer R10.2
- net +3.3V_LDO: now reaches R15.1
- net +3.3V_LDO: now also R16.1, R18.1, R21.1, ASM1.D13 (VCCH), ASM1.D6 (VCCH), ASM1.D8 (VCCH), ASM1.D9 (VCCH), ASM1.E13 (VCCH), ASM1.E6 (VCCH), ASM1.E8 (VCCH), ASM1.E9 (VCCH), ASM1.F13 (VCCH), ASM1.F6 (VCCH), ASM1.H6 (VCCH), ASM2.D13 (VCCH), ASM2.D6 (VCCH), ASM2.D8 (VCCH), ASM2.D9 (VCCH), ASM2.E13 (VCCH), ASM2.E6 (VCCH), ASM2.E8 (VCCH), ASM2.E9 (VCCH), ASM2.F13 (VCCH), ASM2.F6 (VCCH), ASM2.H6 (VCCH), R1.1; no longer PCIe1.A17 (PERn0)
- net USB4_2_SBU1_C: now reaches R13.1
- net USB4_2_SBU1_C: now also USB2.A8 (SBU1); no longer PCIe1.A14 (REFCLK-)
- net USB4_2_2.0_C_D+: now reaches R12.1
- net USB4_2_2.0_C_D+: now also USB2.A6 (D+), USB2.B6 (D+); no longer PCIe1.A13 (REFCLK+)
- net at PCIe1.B17 (~{PRSNT2}), R22.2: now also PCIe1.B31 (~{PRSNT2}), PCIe1.B48 (~{PRSNT2}), PCIe1.B81 (~{PRSNT2})
- net USB4_2_RX1_C-: now reaches USB2.A10 (RX2-)
- net USB4_2_RX1_C-: now also C15.1
- net USB4_2_RX1_C+: now reaches USB2.A11 (RX2+)
- net USB4_2_RX1_C+: now also C16.1
- net USB4_2_TX0_C+: now reaches USB2.A2 (TX1+)
- net USB4_2_TX0_C+: now also C14.1
- net USB4_2_TX0_C-: now reaches USB2.A3 (TX1-)
- net USB4_2_TX0_C-: now also C13.1
- net USB4_2_CC1_C: now reaches USB2.A5 (CC1)
- net USB4_2_CC1_C: now also R9.1
- net USB4_2_2.0_C_D-: now reaches USB2.A7 (D-)
- net USB4_2_2.0_C_D-: now also USB2.B7 (D-)
- net USB4_2_RX0_C-: now reaches USB2.B10 (RX1-)
- net USB4_2_RX0_C+: now reaches USB2.B11 (RX1+)
- net USB4_2_RX0_C+: now also C12.1
- net USB4_2_TX1_C+: now reaches USB2.B2 (TX2+)
- net USB4_2_TX1_C+: now also C18.1
- net USB4_2_TX1_C-: now reaches USB2.B3 (TX2-)
- net USB4_2_TX1_C-: now also C17.1
- net USB4_2_CC2_C: now reaches USB2.B5 (CC2)
- net USB4_2_SBU2_C: now reaches USB2.B8 (SBU2)
- net USB4_2_SBU2_C: now also R14.1
- net PCIe_CLKREQ#: now reaches R22.1
- net PCIe_CLKREQ#: now also R21.2, ASM1.A19 (CLKREQ0#/GPIO8)
- net +3.3V_M.2: now reaches NVME1.10
- net +3.3V_M.2: now also NVME1.12, NVME1.14, NVME1.16, NVME1.18, NVME1.2, NVME1.4
- net M.2_RX1-: now reaches NVME1.29
- net M.2_RX1-: now also ASM2.W20 (PRXN1)
- net M.2_RX1+: now reaches NVME1.31
- net M.2_RX1+: now also ASM2.W21 (PRXP1)
- net at NVME1.35: now also C19.2
- net at NVME1.37: now also C26.2
- net M.2_RX0-: now reaches NVME1.41
- net M.2_RX0-: now also ASM2.N20 (PRXN0)
- net M.2_RX0+: now reaches NVME1.43
- net M.2_RX0+: now also ASM2.N21 (PRXP0)
- net at NVME1.47: now also C27.2
- net at NVME1.49: now also C28.2
- net M.2_PERST#: now reaches NVME1.50
- net M.2_PERST#: now also R17.2, R18.2, ASM2.G21 (PERST0#), C29.2
- net M.2_CLKREQ#: now reaches NVME1.52
- net M.2_CLKREQ#: now also R15.2, ASM2.A19 (CLKREQ0#/GPIO8)
- net M.2_REFCLK-: now reaches NVME1.53
- net M.2_REFCLK-: now also ASM2.Y8 (REFCLKN0)
- net ASM2_PE_WAKE#: now reaches NVME1.54
- net ASM2_PE_WAKE#: now also ASM2.A13 (PE_WAKE#/GPIO22)
- net M.2_REFCLK+: now reaches NVME1.55
- net M.2_REFCLK+: now also ASM2.AA8 (REFCLKP0)
- net PCIe_PERST0#: now reaches PCIe1.A11 (~{PERST})
- net PCIe_PERST0#: now also ASM1.G21 (PERST0#)
- net at PCIe1.B5 (SMCLK): no longer R11.2
- net CC1 renamed USB4_1_CC1
- net USB4_1_CC1: now also ASM1.AA6 (CC1)
- net CC1_C renamed USB4_1_CC1_C
- net CC2 renamed USB4_1_CC2
- net USB4_1_CC2: now also ASM1.Y6 (CC2)
- net CC2_C renamed USB4_1_CC2_C
- net PCIe_PRSNT1 renamed USB4_2_CC1
- net USB4_2_CC1: now also ASM2.AA6 (CC1); no longer PCIe1.A1 (~{PRSNT1})
- net PE_WAKE# renamed ASM1_PE_WAKE#
- net ASM1_PE_WAKE#: now also R16.2, ASM1.A13 (PE_WAKE#/GPIO22), R1.2
- net SBU1 renamed USB4_1_SBU1
- net USB4_1_SBU1: now also ASM1.K1 (SBU1)
- net SBU1_C renamed USB4_1_SBU1_C
- net SBU2 renamed USB4_1_SBU2
- net USB4_1_SBU2: now also ASM1.J1 (SBU2)
- net SBU2_C renamed USB4_1_SBU2_C
- net URX0+ renamed USB4_1_RX0+
- net USB4_1_RX0+: now also ASM1.P1 (URXP0)
- net URX0- renamed USB4_1_RX0-
- net USB4_1_RX0-: now also ASM1.P2 (URXN0)
- net URX0_C+ renamed USB4_1_RX0_C+
- net URX0_C- renamed USB4_1_RX0_C-
- net URX1+ renamed USB4_1_RX1+
- net USB4_1_RX1+: now also ASM1.Y2 (URXP1)
- net URX1- renamed USB4_1_RX1-
- net USB4_1_RX1-: now also ASM1.Y1 (URXN1)
- net URX1_C+ renamed USB4_1_RX1_C+
- net URX1_C- renamed USB4_1_RX1_C-
- net USB2_C_D+ renamed USB4_1_2.0_C_D+
- net USB2_C_D- renamed USB4_1_2.0_C_D-
- net USB2_D+ renamed USB4_1_2.0_D+
- net USB4_1_2.0_D+: now also ASM1.M1 (UDP)
- net USB2_D- renamed USB4_1_2.0_D-
- net USB4_1_2.0_D-: now also ASM1.M2 (UDM)
- net UTX0+ renamed USB4_1_TX0+
- net USB4_1_TX0+: now also ASM1.T1 (UTXP0)
- net UTX0- renamed USB4_1_TX0-
- net USB4_1_TX0-: now also ASM1.T2 (UTXN0)
- net UTX0_C+ renamed USB4_1_TX0_C+
- net UTX0_C- renamed USB4_1_TX0_C-
- net UTX1+ renamed USB4_1_TX1+
- net USB4_1_TX1+: now also ASM1.V2 (UTXP1)
- net UTX1- renamed USB4_1_TX1-
- net USB4_1_TX1-: now also ASM1.V1 (UTXN1)
- net UTX1_C+ renamed USB4_1_TX1_C+
- net UTX1_C- renamed USB4_1_TX1_C-
- net XI renamed USB4_2_RX0-
- net USB4_2_RX0-: now also ASM2.P2 (URXN0)
- new net: USB6.A1 (GND), USB6.A12 (GND), USB6.B1 (GND), USB6.B12 (GND)
- new net: USB6.A4 (VBUS), USB6.A9 (VBUS), USB6.B4 (VBUS), USB6.B9 (VBUS)
- new net +3.3VA: ASM1.H5 (VCCA33), ASM2.H5 (VCCA33)
- new net ASM1_ActLED1: ASM1.D1 (NVMeACTLED1/GPIO0)
- new net ASM1_ActLED2: ASM1.A1 (NVMeACTLED2/GPIO3)
- new net ASM1_ActLED3: ASM1.A16 (NVMeACTLED3/GPIO25)
- new net ASM1_ActLED4: ASM1.A17 (NVMeACTLED4/GPIO26)
- new net ASM1_CLKREQ1#: ASM1.A20 (CLKREQ1#/GPIO14)
- new net ASM1_CLKREQ2#: ASM1.A14 (CLKREQ2#/GPIO23)
- new net ASM1_CLKREQ3#: ASM1.A15 (CLKREQ3#/GPIO24)
- new net ASM1_GPIO1: ASM1.C1 (I2C_INT/GPIO1)
- new net ASM1_GPIO19: ASM1.A10 (PRSNT1#/GPIO19)
- new net ASM1_GPIO2: ASM1.B1 (PRSNT#/GPIO2)
- new net ASM1_GPIO20: ASM1.A11 (HDDPC1/GPIO20)
- new net ASM1_GPIO21: ASM1.A12 (PRSNT2#/GPIO21)
- new net ASM1_GPIO27: ASM1.A18 (PRSNT3#/GPIO27)
- new net ASM1_P1_LED: ASM1.A6 (P1_LED/GPIO15)
- new net ASM1_P2_LED: ASM1.A7 (P2_LED/GPIO16)
- new net ASM1_P3_LED: ASM1.A8 (P3_LED/GPIO17)
- new net ASM1_P4_LED: ASM1.A9 (P4_LED/GPIO18)
- new net ASM1_RST#: ASM1.H1 (RST#)
- new net ASM1_SPI_CLK: ASM1.A5 (GPIO6/SPI_CLK)
- new net ASM1_SPI_CS#: ASM1.A2 (GPIO4/SPI_CS#)
- new net ASM1_SPI_DI: ASM1.A4 (GPIO7/SPI_DI)
- new net ASM1_SPI_DO: ASM1.A3 (GPIO5/SPI_DO)
- new net ASM1_TEST_EN: ASM1.H21 (TEST_EN)
- new net ASM1_UREXT: ASM1.AA3 (REXT)
- new net ASM1_VBUS: ASM1.G1 (VBUS)
- new net ASM1_XI: ASM1.AA4 (XI)
- new net ASM1_XO: ASM1.Y4 (XO)
- new net ASM2_ActLED1: ASM2.D1 (NVMeACTLED1/GPIO0)
- new net ASM2_ActLED2: ASM2.A1 (NVMeACTLED2/GPIO3)
- new net ASM2_ActLED3: ASM2.A16 (NVMeACTLED3/GPIO25)
- new net ASM2_ActLED4: ASM2.A17 (NVMeACTLED4/GPIO26)
- new net ASM2_CLKREQ2#: ASM2.A14 (CLKREQ2#/GPIO23)
- new net ASM2_CLKREQ3#: ASM2.A15 (CLKREQ3#/GPIO24)
- new net ASM2_GPIO1: ASM2.C1 (I2C_INT/GPIO1)
- new net ASM2_GPIO19: ASM2.A10 (PRSNT1#/GPIO19)
- new net ASM2_GPIO2: ASM2.B1 (PRSNT#/GPIO2)
- new net ASM2_GPIO20: ASM2.A11 (HDDPC1/GPIO20)
- new net ASM2_GPIO21: ASM2.A12 (PRSNT2#/GPIO21)
- new net ASM2_GPIO27: ASM2.A18 (PRSNT3#/GPIO27)
- new net ASM2_HDDPC: ASM2.C21 (HDDPC)
- new net ASM2_P1_LED: ASM2.A6 (P1_LED/GPIO15)
- new net ASM2_P2_LED: ASM2.A7 (P2_LED/GPIO16)
- new net ASM2_P3_LED: ASM2.A8 (P3_LED/GPIO17)
- new net ASM2_P4_LED: ASM2.A9 (P4_LED/GPIO18)
- new net ASM2_RST#: ASM2.H1 (RST#)
- new net ASM2_SPI_CLK: ASM2.A5 (GPIO6/SPI_CLK)
- new net ASM2_SPI_CS#: ASM2.A2 (GPIO4/SPI_CS#)
- new net ASM2_SPI_DI: ASM2.A4 (GPIO7/SPI_DI)
- new net ASM2_SPI_DO: ASM2.A3 (GPIO5/SPI_DO)
- new net ASM2_TEST_EN: ASM2.H21 (TEST_EN)
- new net ASM2_UREXT: ASM2.AA3 (REXT)
- new net ASM2_XI: ASM2.AA4 (XI)
- new net ASM2_XO: ASM2.Y4 (XO)
- new net GNDA: ASM1.AA1 (GNDA), ASM1.AA12 (GNDA), ASM1.AA14 (GNDA), ASM1.AA16 (GNDA), ASM1.AA18 (GNDA), ASM1.AA2 (GNDA), ASM1.AA20 (GNDA), ASM1.AA21 (GNDA), ASM1.AA5 (GNDA), ASM1.AA9 (GNDA), ASM1.L1 (GNDA), ASM1.L2 (GNDA), ASM1.L4 (GNDA), ASM1.L5 (GNDA), ASM1.M20 (GNDA), ASM1.M21 (GNDA), ASM1.N1 (GNDA), ASM1.N17 (GNDA), ASM1.N18 (GNDA), ASM1.N2 (GNDA), ASM1.N4 (GNDA), ASM1.N5 (GNDA), ASM1.P17 (GNDA), ASM1.P18 (GNDA), ASM1.P20 (GNDA), ASM1.P21 (GNDA), ASM1.P4 (GNDA), ASM1.P5 (GNDA), ASM1.R1 (GNDA), ASM1.R2 (GNDA), ASM1.T17 (GNDA), ASM1.T18 (GNDA), ASM1.T20 (GNDA), ASM1.T21 (GNDA), ASM1.T4 (GNDA), ASM1.T5 (GNDA), ASM1.U1 (GNDA), ASM1.U17 (GNDA), ASM1.U18 (GNDA), ASM1.U2 (GNDA), ASM1.U4 (GNDA), ASM1.U5 (GNDA), ASM1.V11 (GNDA), ASM1.V13 (GNDA), ASM1.V14 (GNDA), ASM1.V16 (GNDA), ASM1.V17 (GNDA), ASM1.V18 (GNDA), ASM1.V20 (GNDA), ASM1.V21 (GNDA), ASM1.V4 (GNDA), ASM1.V5 (GNDA), ASM1.V6 (GNDA), ASM1.V8 (GNDA), ASM1.V9 (GNDA), ASM1.W1 (GNDA), ASM1.W2 (GNDA), ASM1.Y12 (GNDA), ASM1.Y14 (GNDA), ASM1.Y16 (GNDA), ASM1.Y18 (GNDA), ASM1.Y20 (GNDA), ASM1.Y21 (GNDA), ASM1.Y3 (GNDA), ASM1.Y5 (GNDA), ASM1.Y9 (GNDA), ASM2.AA1 (GNDA), ASM2.AA12 (GNDA), ASM2.AA14 (GNDA), ASM2.AA16 (GNDA), ASM2.AA18 (GNDA), ASM2.AA2 (GNDA), ASM2.AA20 (GNDA), ASM2.AA21 (GNDA), ASM2.AA5 (GNDA), ASM2.AA9 (GNDA), ASM2.L1 (GNDA), ASM2.L2 (GNDA), ASM2.L4 (GNDA), ASM2.L5 (GNDA), ASM2.M20 (GNDA), ASM2.M21 (GNDA), ASM2.N1 (GNDA), ASM2.N17 (GNDA), ASM2.N18 (GNDA), ASM2.N2 (GNDA), ASM2.N4 (GNDA), ASM2.N5 (GNDA), ASM2.P17 (GNDA), ASM2.P18 (GNDA), ASM2.P20 (GNDA), ASM2.P21 (GNDA), ASM2.P4 (GNDA), ASM2.P5 (GNDA), ASM2.R1 (GNDA), ASM2.R2 (GNDA), ASM2.T17 (GNDA), ASM2.T18 (GNDA), ASM2.T20 (GNDA), ASM2.T21 (GNDA), ASM2.T4 (GNDA), ASM2.T5 (GNDA), ASM2.U1 (GNDA), ASM2.U17 (GNDA), ASM2.U18 (GNDA), ASM2.U2 (GNDA), ASM2.U4 (GNDA), ASM2.U5 (GNDA), ASM2.V11 (GNDA), ASM2.V13 (GNDA), ASM2.V14 (GNDA), ASM2.V16 (GNDA), ASM2.V17 (GNDA), ASM2.V18 (GNDA), ASM2.V20 (GNDA), ASM2.V21 (GNDA), ASM2.V4 (GNDA), ASM2.V5 (GNDA), ASM2.V6 (GNDA), ASM2.V8 (GNDA), ASM2.V9 (GNDA), ASM2.W1 (GNDA), ASM2.W2 (GNDA), ASM2.Y12 (GNDA), ASM2.Y14 (GNDA), ASM2.Y16 (GNDA), ASM2.Y18 (GNDA), ASM2.Y20 (GNDA), ASM2.Y21 (GNDA), ASM2.Y3 (GNDA), ASM2.Y5 (GNDA), ASM2.Y9 (GNDA)
- new net M.2_TX0+: ASM2.R20 (PTXP0), C28.1
- new net M.2_TX0-: ASM2.R21 (PTXN0), C27.1
- new net M.2_TX1+: ASM2.U20 (PTXP1), C26.1
- new net M.2_TX1-: ASM2.U21 (PTXN1), C19.1
- new net PCIe_HDDPC: ASM1.C21 (HDDPC)
- new net SW_CLKREQ#: ASM2.A20 (CLKREQ1#/GPIO14)
- new net SW_PERST#: ASM2.E21 (NC/PERST2#)
- new net SW_REFCLK+: ASM2.AA10 (NC/REFCLKP2)
- new net SW_REFCLK-: ASM2.Y10 (NC/REFCLKN2)
- new net SW_RX0+: ASM2.Y19 (PRXP2)
- new net SW_RX0-: ASM2.AA19 (PRXN2)
- new net SW_RX1+: ASM2.AA13 (PRXP3)
- new net SW_RX1-: ASM2.Y13 (PRXN3)
- new net SW_TX0+: ASM2.Y17 (PTXP2)
- new net SW_TX0-: ASM2.AA17 (PTXN2)
- new net SW_TX1+: ASM2.Y15 (PTXP3)
- new net SW_TX1-: ASM2.AA15 (PTXN3)
- new net USB4_2_2.0_D+: ASM2.M1 (UDP), R12.2
- new net USB4_2_2.0_D-: ASM2.M2 (UDM), R11.2
- new net USB4_2_CC2: ASM2.Y6 (CC2), R10.2
- new net USB4_2_RX0+: ASM2.P1 (URXP0), C12.2
- new net USB4_2_RX1+: ASM2.Y2 (URXP1), C16.2
- new net USB4_2_RX1-: ASM2.Y1 (URXN1), C15.2
- new net USB4_2_SBU1: ASM2.K1 (SBU1), R13.2
- new net USB4_2_SBU2: ASM2.J1 (SBU2), R14.2
- new net USB4_2_TX0+: ASM2.T1 (UTXP0), C14.2
- new net USB4_2_TX0-: ASM2.T2 (UTXN0), C13.2
- new net USB4_2_TX1+: ASM2.V2 (UTXP1), C18.2
- new net USB4_2_TX1-: ASM2.V1 (UTXN1), C17.2
- new net VCCL: ASM1.L16 (VCCL), ASM1.L17 (VCCL), ASM1.L18 (VCCL), ASM1.L20 (VCCL), ASM1.L21 (VCCL), ASM1.L6 (VCCL), ASM1.N16 (VCCL), ASM1.N6 (VCCL), ASM1.P16 (VCCL), ASM1.P6 (VCCL), ASM1.T16 (VCCL), ASM1.T6 (VCCL), ASM1.U11 (VCCL), ASM1.U13 (VCCL), ASM1.U14 (VCCL), ASM1.U16 (VCCL), ASM1.U6 (VCCL), ASM2.L16 (VCCL), ASM2.L17 (VCCL), ASM2.L18 (VCCL), ASM2.L20 (VCCL), ASM2.L21 (VCCL), ASM2.L6 (VCCL), ASM2.N16 (VCCL), ASM2.N6 (VCCL), ASM2.P16 (VCCL), ASM2.P6 (VCCL), ASM2.T16 (VCCL), ASM2.T6 (VCCL), ASM2.U11 (VCCL), ASM2.U13 (VCCL), ASM2.U14 (VCCL), ASM2.U16 (VCCL), ASM2.U6 (VCCL)
- new net VDD: ASM1.D14 (VDD), ASM1.D16 (VDD), ASM1.E11 (VDD), ASM1.E14 (VDD), ASM1.E16 (VDD), ASM1.F11 (VDD), ASM1.F14 (VDD), ASM1.F16 (VDD), ASM1.F9 (VDD), ASM1.H11 (VDD), ASM1.H13 (VDD), ASM1.H14 (VDD), ASM1.H16 (VDD), ASM1.H9 (VDD), ASM1.J13 (VDD), ASM1.J14 (VDD), ASM1.J16 (VDD), ASM1.J17 (VDD), ASM1.J18 (VDD), ASM1.J20 (VDD), ASM1.J21 (VDD), ASM1.J8 (VDD), ASM1.J9 (VDD), ASM1.K20 (VDD), ASM1.K21 (VDD), ASM1.L11 (VDD), ASM1.L14 (VDD), ASM1.L8 (VDD), ASM1.N14 (VDD), ASM1.N8 (VDD), ASM1.P13 (VDD), ASM1.P14 (VDD), ASM1.P8 (VDD), ASM1.T11 (VDD), ASM1.T13 (VDD), ASM1.T14 (VDD), ASM1.T8 (VDD), ASM1.T9 (VDD), ASM1.U8 (VDD), ASM1.U9 (VDD), ASM2.D14 (VDD), ASM2.D16 (VDD), ASM2.E11 (VDD), ASM2.E14 (VDD), ASM2.E16 (VDD), ASM2.F11 (VDD), ASM2.F14 (VDD), ASM2.F16 (VDD), ASM2.F9 (VDD), ASM2.H11 (VDD), ASM2.H13 (VDD), ASM2.H14 (VDD), ASM2.H16 (VDD), ASM2.H9 (VDD), ASM2.J13 (VDD), ASM2.J14 (VDD), ASM2.J16 (VDD), ASM2.J17 (VDD), ASM2.J18 (VDD), ASM2.J20 (VDD), ASM2.J21 (VDD), ASM2.J8 (VDD), ASM2.J9 (VDD), ASM2.K20 (VDD), ASM2.K21 (VDD), ASM2.L11 (VDD), ASM2.L14 (VDD), ASM2.L8 (VDD), ASM2.N14 (VDD), ASM2.N8 (VDD), ASM2.P13 (VDD), ASM2.P14 (VDD), ASM2.P8 (VDD), ASM2.T11 (VDD), ASM2.T13 (VDD), ASM2.T14 (VDD), ASM2.T8 (VDD), ASM2.T9 (VDD), ASM2.U8 (VDD), ASM2.U9 (VDD)
- no-connect marks 41 -> 172
Other:
- moved on the sheet: NVME1, USB1

Commit message: clean up
Parts:
- removed U1: PCI11414-I/PMX, easyeda2kicad:QFN-164_L13.0-W13.0-P0.50-TL-EP8.0, symbol easyeda2kicad:PCI11414-I_PMX
- added C30, C31, C32, C33: 0.1u, Capacitor_SMD:C_0402_1005Metric, symbol Device:C_Small
- added R19, R20: 49.9Ω, Resistor_SMD:R_0402_1005Metric, symbol Device:R_Small
- added U1: PCI11414 DQFN-164, symbol egpulib:PCI11414 DQFN-164
Connections:
- net +3.3V_M.2: now also NVME1.70, NVME1.72, NVME1.74
- net ASM2_TEST_EN: now also U1.127 (TESTEN)
- net GND: now also R19.1, R20.1, U1.125 (ATEST0)
- net SW_PERST#: now also U1.128 (PCIE_PERST_N)
- net SW_REFCLK+: now also R19.2, U1.145 (PCIE_REFCLK_IN_P)
- net SW_REFCLK-: now also R20.2, U1.146 (PCIE_REFCLK_IN_M)
- net SW_RX0+: now also U1.12 (PCIE_RXP_L0_P0)
- net SW_RX0-: now also U1.13 (PCIE_RXM_L0_P0)
- net SW_RX1+: now also U1.27 (PCIE_RXP_L1_P0)
- net SW_RX1-: now also U1.26 (PCIE_RXM_L1_P0)
- net SW_TX0+: now also C31.1
- net SW_TX0-: now also C30.1
- net SW_TX1+: now also C33.1
- net SW_TX1-: now also C32.1
- new net: C31.2, U1.16 (PCIE_TXP_L0_P0)
- new net: C33.2, U1.23 (PCIE_TXP_L1_P0)
- new net: C30.2, U1.17 (PCIE_TXM_L0_P0)
- new net: C32.2, U1.22 (PCIE_TXM_L1_P0)
- no-connect marks 172 -> 183
Other:
- moved on the sheet: U3
