File: eGPU-dock/GPU1.kicad_sch (KiCad schematic)
At the start: 151 parts, among them CON1 USB_C_Plug, J1 Conn_01x04, J2 Conn_01x02, J3 Conn_01x02, J4 Conn_01x04, SW1 SW_Push, SW2 SW_Push, SW3 SW_Push, SW4 SW_Push, U3 W25X20CLSN, X1 25 Mhz

Commit message: almost as masive schematic update
Parts:
- added C74, C75: 0UF, Capacitor_SMD:C_0402_1005Metric, symbol Device:C
- added L1: L, symbol Device:L
- added R10, R12, R15, R16, R18, R3, R5, R7, R76, R77, R78, R8, R9: 0Ω, Resistor_SMD:R_0402_1005Metric, symbol Device:R
- added R45, R47, R49, R51, R52, R53, R56, R58: 4.7KΩ, Resistor_SMD:R_0402_1005Metric, symbol Device:R
- added T1, T10, T11, T2, T3, T4, T5, T6, T7, T8, T9: TestPoint, TestPoint:TestPoint_Pad_1.0x1.0mm, symbol Connector:TestPoint
- FB1: footprint (none) -> Inductor_SMD:L_0402_1005Metric
Connections:
- net GND: now also R45.2, R47.2, R49.2, R51.2, R52.2, R53.2, R56.2, R58.2
- net GPIO14: now also R45.1, T4.1
- net GPIO19: now also R47.1, T5.1
- net GPIO20: now also R49.1, T6.1
- net GPIO21: now also R51.1, T7.1
- net GPIO22: now also R52.1
- net GPIO23: now also R53.1, T9.1
- net GPIO24: now also R56.1, T10.1
- net GPIO27: now also R58.1, T11.1
- net PERST_B1: now also T1.1
- net PERST_B3: now also T2.1
- net UART_RX: now also T3.1
- net VCC18: now also ASM1.L16 (VCCL), ASM1.L17 (VCCL), ASM1.L18 (VCCL), ASM1.L20 (VCCL), ASM1.L21 (VCCL), ASM1.L6 (VCCL), ASM1.N16 (VCCL), ASM1.N6 (VCCL), ASM1.P16 (VCCL), ASM1.P6 (VCCL), ASM1.T16 (VCCL), ASM1.T6 (VCCL), ASM1.U11 (VCCL), ASM1.U13 (VCCL), ASM1.U14 (VCCL), ASM1.U16 (VCCL), ASM1.U6 (VCCL)
- net VCC33_SYS: now also ASM1.D13 (VCCH), ASM1.D6 (VCCH), ASM1.D8 (VCCH), ASM1.D9 (VCCH), ASM1.E13 (VCCH), ASM1.E6 (VCCH), ASM1.E8 (VCCH), ASM1.E9 (VCCH), ASM1.F13 (VCCH), ASM1.F6 (VCCH), ASM1.H6 (VCCH)
- net VCCA33: now also ASM1.H5 (VCCA33)
Other:
- note added: "EX. TIXX988"
- note added: "Place holders"
- note added: "To power delivery chip"
- moved on the sheet: ASM1E, J1, R34, R42
