File: eGPU-dock/GPU2.kicad_sch (KiCad schematic)
At the start: 0 parts

Commit message: almost as masive schematic update
Parts:
- added ATXPWR1: ATX-24, symbol Connector:ATX-24
- added C100, C95, C96, C99: 22UF/10V, Capacitor_SMD:C_0402_1005Metric, symbol Device:C
- added C101, C105, C156, C81, C82, C84, C85, C92, C93: 0.1UF/16V, Capacitor_SMD:C_0402_1005Metric, symbol Device:C
- added C102, C106: 3300PF/50V, Capacitor_SMD:C_0402_1005Metric, symbol Device:C
- added C103, C104, C97, C98: 10UF/25V, Capacitor_SMD:C_0402_1005Metric, symbol Device:C
- added C76, C77: 15PF/50V, Capacitor_SMD:C_0402_1005Metric, symbol Device:C
- added C78, C79: 22UF/6.3V, Capacitor_SMD:C_0402_1005Metric, symbol Device:C
- added C80, C83: 10UF/16V, Capacitor_SMD:C_0402_1005Metric, symbol Device:C
- added C88, C89: 2.2UF/6.3V, Capacitor_SMD:C_0402_1005Metric, symbol Device:C
- added C91, C94: 0.1UF/50V, Capacitor_SMD:C_0402_1005Metric, symbol Device:C
- added D10, D11: SR34, Diode_SMD:D_SMB, symbol Device:D_Schottky
- added D12, D13: B130LAW, Diode_SMD:Nexperia_CFP3_SOD-123W, symbol Device:D_Schottky
- added J21, J22, J23, J24, J25, J6, J7: Conn_01x02, Connector_PinHeader_2.54mm:PinHeader_1x02_P2.54mm_Vertical, symbol Connector_Generic:Conn_01x02
- added L2, L3: 2.2UH, Inductor_SMD:L_0402_1005Metric, symbol Device:L
- added L4, L5: 10UH, Inductor_SMD:L_0402_1005Metric, symbol Device:L
- added LED10: LED, symbol Device:LED
- added Q1: GS1117AXF, Package_TO_SOT_SMD:SOT-223, symbol egpulib:GS1117AXF
- added R1: 2.2KΩ, Resistor_SMD:R_0402_1005Metric, symbol Device:R
- added R100, R103, R81, R85: 100KΩ, Resistor_SMD:R_0402_1005Metric, symbol Device:R
- added R101, R104, R105, R107, R75, R84, R93, R94, R95, R96, R97, R99: 0Ω, Resistor_SMD:R_0402_1005Metric, symbol Device:R
- added R102: 51KΩ, Resistor_SMD:R_0402_1005Metric, symbol Device:R
- added R106, R108: 10KΩ, Resistor_SMD:R_0402_1005Metric, symbol Device:R
- added R109, R110: 7.5KΩ, Resistor_SMD:R_0402_1005Metric, symbol Device:R
- added R111: 1KΩ, Resistor_SMD:R_0402_1005Metric, symbol Device:R
- added R79: 330KΩ, Resistor_SMD:R_0402_1005Metric, symbol Device:R
- added R80, R89: 150KΩ, Resistor_SMD:R_0402_1005Metric, symbol Device:R
- added R82: 165Ω, Resistor_SMD:R_0402_1005Metric, symbol Device:R
- added R83: 100Ω, Resistor_SMD:R_0402_1005Metric, symbol Device:R
- added R90: 180KΩ, Resistor_SMD:R_0402_1005Metric, symbol Device:R
- added R98: 28KΩ, Resistor_SMD:R_0402_1005Metric, symbol Device:R
- added U1, U8: MP2307DN, Package_SO:SOIC-8-1EP_3.9x4.9mm_P1.27mm_EP2.29x3mm, symbol egpulib:MP2307
- added U5: RT8059, Package_TO_SOT_SMD:TSOT-23-5, symbol egpulib:RT8059
- added U6: ID8225B-ADA60, Package_TO_SOT_SMD:SOT-23-6, symbol egpulib:ID8225B
Connections:
- new net: R102.2, R108.1, U8.5 (FB)
- new net: C106.1, R110.2
- new net: C105.2, C106.2, U8.6 (COMP)
- new net: C97.2, C98.2, R104.2, R94.2, R95.2, U1.2 (IN)
- new net: LED10.1 (K), R111.1
- new net: R106.1, R98.2, U1.5 (FB)
- new net: D10.1 (K), J6.2 (Pin_2), R96.2, R97.2
- new net: R80.2, R90.1, U6.6 (FB)
- new net: C102.1, R109.2
- new net: L2.1, U5.3 (SW)
- new net: C101.2, C102.2, U1.6 (COMP)
- new net: C94.2, U8.1 (BS)
- new net: C92.1, U1.8 (SS)
- new net: D11.1 (K), J7.2 (Pin_2), R101.2, R99.2
- new net: L3.1, U6.3 (SW)
- new net: C93.1, U8.8 (SS)
- new net: C91.2, U1.1 (BS)
- new net +1.05V_EN: C85.2, R81.2, U6.1 (EN)
- new net +1.05V_PG: R75.1, U6.5 (PG)
- new net +12V: J24.1 (Pin_1)
- new net +12V_AD: C103.2, C104.2, J23.1 (Pin_1), R103.1, R104.1, U8.2 (IN)
- new net +12V_ATX: ATXPWR1.10 (+12V), ATXPWR1.11 (+12V), J23.2 (Pin_2), J24.2 (Pin_2)
- new net +3.3V: J25.1 (Pin_1), J6.1 (Pin_1), J7.1 (Pin_1)
- new net +3.3V_ATX: ATXPWR1.1 (+3.3V), ATXPWR1.12 (+3.3V), ATXPWR1.13 (+3.3V), ATXPWR1.2 (+3.3V), J21.1 (Pin_1)
- new net +5V_ATX: ATXPWR1.21 (+5V), ATXPWR1.22 (+5V), ATXPWR1.23 (+5V), ATXPWR1.4 (+5V), ATXPWR1.6 (+5V), J25.2 (Pin_2)
- new net +5V_BUS: C82.2, C83.2, C88.2, C89.2, Q1.3 (IN), R81.1, R85.1, R95.1, U5.4 (VIN), U6.4 (VIN)
- new net +5V_BUS_CON: R94.1
- new net +5V_SB: ATXPWR1.9 (+5VSB), R1.1
- new net -12V_ATX: ATXPWR1.14 (-12V)
- new net 1V8_EN: C84.2, R85.2, U5.1 (EN)
- new net 3V3OUT_1D: C80.2, C81.2, Q1.2 (OUT), Q1.4 (Vout), R83.1, R84.2
- new net 5V_AD: C100.2, C99.2, D11.2 (A), L5.2, LED10.2 (A), R101.1, R102.1, R99.1
- new net AD2: C95.2, C96.2, D10.2 (A), L4.2, R96.1, R97.1, R98.1
- new net FB_1V8: C77.1, R79.2, R89.1, U5.5 (OUT)
- new net FB_3V3_1D: Q1.1 (ADJ/GND), R82.1, R83.2
- new net GND: ATXPWR1.15 (GND), ATXPWR1.17 (GND), ATXPWR1.18 (GND), ATXPWR1.19 (GND), ATXPWR1.24 (GND), ATXPWR1.3 (GND), ATXPWR1.5 (GND), ATXPWR1.7 (GND), C100.1, C101.1, C103.1, C104.1, C105.1, C156.1, C76.1, C78.1, C79.1, C80.1, C81.1, C82.1, C83.1, C84.1, C85.1, C88.1, C89.1, C92.2, C93.2, C95.1, C96.1, C97.1, C98.1, C99.1, D12.2 (A), D13.2 (A), J22.2 (Pin_2), R105.2, R106.2, R107.2, R108.2, R109.1, R110.1, R111.2, R82.2, R89.2, R90.2, U1.4 (GND1), U1.9 (GND2), U5.2 (GND), U6.2 (GND), U8.4 (GND1), U8.9 (GND2)
- new net HDDPC_C: R93.2
- new net MP2307_EN: R100.2, R103.2, R105.1, R107.1, R93.1, U1.7 (EN), U8.7 (EN)
- new net PS_ON#: ATXPWR1.16 (PS_ON#), C156.2, J22.1 (Pin_1), R1.2
- new net RST: R75.2
- new net VCC18: C77.2, C78.2, L2.2, R79.1
- new net VCC33_SYS: J21.2 (Pin_2), R100.1, R84.1
- new net VDD095: C76.2, C79.2, L3.2, R80.1
- new net VMAIN_LX: C94.1, D13.1 (K), L5.1, U8.3 (SW)
- new net VMAIN_LX__3V: C91.1, D12.1 (K), L4.1, U1.3 (SW)
- no-connect marks 0 -> 1
Other:
- note added: "0.925(1+R1/R2)=VOUT 44.2K:10K=5V 26.1K:10K=3.3V 28K:10K=3.5V 47K:10K=5.27V 47.5K:10K=5.32V 48.7K:10K=5.43V 51K:10K=5.64V"
- note added: "0.925(1+R1/R2)=VOUT 44.2K:10K=5V 26.1K:10K=3.3V 47K:10K=5.27V 47.5K:10K=5.32V 48.7K:10K=5.43V"
- note added: "1.074V=0.6(1+158k/180k)"
- note added: "1.92=0.6(1+330K/150K)"
- note added: "1A"
- note added: "3.3V=1.25(1+165/100)"
- note added: "3A"
- note added: "51K:10K=5.64V"
- note added: "For PCIe device"
- note added: "HDDPC 3.3V tolerance"
- note added: "Power 3.3V for ASM2464PDX and TI PDC 8mA (GS1117AXF)"
- note added: "R1"
- note added: "R2"
- note added: "Vout=0.6(1+R1/R2) , 1.8=0.6(1+300K/150K)"
- note added: "Vout=0.6(1+R1/R2) 1.01V=0.6(1+150k/220k), 1.1V=0.6(1+150k/180k)"
- note added: "Vout=1.25(1+R2/R1)"
- note added: "power on"
- note added: "self power"
